Commit message: ignitona geçiş denemesi (bozuk)

File: robotaksi_description/urdf/d435_camera.xacro (robot description, xacro)
@@ -87,5 +87,4 @@
     <!-- RGB Camera Gazebo Plugin -->
     <gazebo reference="${name}_color_frame">
-      <material>Gazebo/DarkGrey</material>
       <sensor name="${name}_rgb_camera" type="camera">
         <pose>0 0 0 0 0 0</pose>
@@ -110,18 +109,10 @@
         <update_rate>30</update_rate>
         <visualize>true</visualize>
-        <plugin name="${name}_rgb_camera_controller" filename="libgazebo_ros_camera.so">
-          <ros>
-            <namespace>/</namespace>
-          </ros>
-          <camera_name>${name}_rgb</camera_name>
-          <frame_name>${name}_color_optical_frame</frame_name>
-          <image_topic_name>camera/color/image_raw</image_topic_name>
-          <camera_info_topic_name>camera/color/camera_info</camera_info_topic_name>
-        </plugin>
+        <topic>/camera/color/image_raw</topic>
+        <camera_info_topic>/camera/color/camera_info</camera_info_topic>
       </sensor>
     </gazebo>
-    <!-- Depth Camera Gazebo Plugin -->
     <gazebo reference="${name}_depth_frame">
-      <sensor name="${name}_depth_camera" type="depth">
+      <sensor name="${name}_depth_camera" type="depth_camera">
         <pose>0 0 0 0 0 0</pose>
         <camera>
@@ -145,45 +136,9 @@
         <update_rate>30</update_rate>
         <visualize>false</visualize>
-        <plugin name="${name}_depth_camera_controller" filename="libgazebo_ros_camera.so">
-          <ros>
-            <namespace>/</namespace>
-          </ros>
-          <camera_name>${name}_depth</camera_name>
-          <frame_name>${name}_depth_optical_frame</frame_name>
-          <image_topic_name>camera/depth/image_raw</image_topic_name>
-          <camera_info_topic_name>camera/depth/camera_info</camera_info_topic_name>
-        </plugin>
-      </sensor>
-    </gazebo>
-    <!-- Point Cloud Plugin -->
-    <gazebo reference="${name}_depth_frame">
-      <sensor name="${name}_pointcloud" type="depth">
-        <pose>0 0 0 0 0 0</pose>
-        <camera>
-          <horizontal_fov>1.047</horizontal_fov>
-          <image>
-            <width>640</width>
-            <height>480</height>
-          </image>
-          <clip>
-            <near>0.1</near>
-            <far>10.0</far>
-          </clip>
-        </camera>
-        <always_on>1</always_on>
-        <update_rate>15</update_rate>
-        <visualize>false</visualize>
-        <plugin name="${name}_pointcloud_controller" filename="libgazebo_ros_depth_camera.so">
-          <ros>
-            <namespace>/</namespace>
-          </ros>
-          <camera_name>${name}_points</camera_name>
-          <frame_name>${name}_depth_optical_frame</frame_name>
-          <point_cloud_topic_name>camera/depth/color/points</point_cloud_topic_name>
-          <image_topic_name>camera/depth/image_rect_raw</image_topic_name>
-          <camera_info_topic_name>camera/depth/camera_info</camera_info_topic_name>
-          <point_cloud_cutoff>0.1</point_cloud_cutoff>
-          <point_cloud_cutoff_max>10.0</point_cloud_cutoff_max>
-        </plugin>
+        <topic>/camera/depth/image_raw</topic>
+        <camera_info_topic>/camera/depth/camera_info</camera_info_topic>
+        <point_cloud>
+          <topic>/camera/depth/color/points</topic>
+        </point_cloud>
       </sensor>
     </gazebo>

File: robotaksi_description/urdf/imu.xacro (robot description, xacro)
@@ -28,65 +28,5 @@
         <update_rate>100</update_rate>
         <visualize>true</visualize>
-        <plugin name="${name}_plugin" filename="libgazebo_ros_imu_sensor.so">
-          <ros>
-            <namespace>/</namespace>
-            <remapping>~/out:=imu/data</remapping>
-          </ros>
-          <initial_orientation_as_reference>false</initial_orientation_as_reference>
-        </plugin>
-        <imu>
-          <angular_velocity>
-            <x>
-              <noise type="gaussian">
-                <mean>0.0</mean>
-                <stddev>2e-4</stddev>
-                <bias_mean>0.0000075</bias_mean>
-                <bias_stddev>0.0000008</bias_stddev>
-              </noise>
-            </x>
-            <y>
-              <noise type="gaussian">
-                <mean>0.0</mean>
-                <stddev>2e-4</stddev>
-                <bias_mean>0.0000075</bias_mean>
-                <bias_stddev>0.0000008</bias_stddev>
-              </noise>
-            </y>
-            <z>
-              <noise type="gaussian">
-                <mean>0.0</mean>
-                <stddev>2e-4</stddev>
-                <bias_mean>0.0000075</bias_mean>
-                <bias_stddev>0.0000008</bias_stddev>
-              </noise>
-            </z>
-          </angular_velocity>
-          <linear_acceleration>
-            <x>
-              <noise type="gaussian">
-                <mean>0.0</mean>
-                <stddev>1.7e-2</stddev>
-                <bias_mean>0.1</bias_mean>
-                <bias_stddev>0.001</bias_stddev>
-              </noise>
-            </x>
-            <y>
-              <noise type="gaussian">
-                <mean>0.0</mean>
-                <stddev>1.7e-2</stddev>
-                <bias_mean>0.1</bias_mean>
-                <bias_stddev>0.001</bias_stddev>
-              </noise>
-            </y>
-            <z>
-              <noise type="gaussian">
-                <mean>0.0</mean>
-                <stddev>1.7e-2</stddev>
-                <bias_mean>0.1</bias_mean>
-                <bias_stddev>0.001</bias_stddev>
-              </noise>
-            </z>
-          </linear_acceleration>
-        </imu>
+        <topic>/imu/data</topic>
       </sensor>
     </gazebo>

File: robotaksi_description/urdf/robotaksi.xacro (robot description, xacro)
@@ -1,4 +1,6 @@
 <?xml version="1.0" ?>
 <robot name="robotaksi" xmlns:xacro="http://www.ros.org/wiki/xacro">
+<xacro:arg name="is_sim" default="true"/>
+<xacro:arg name="is_ignition" default="true"/>
 <xacro:include filename="$(find robotaksi_description)/urdf/materials.xacro" />
 <xacro:include filename="$(find robotaksi_description)/urdf/robotaksi.gazebo" />
@@ -190,8 +192,20 @@
   <axis xyz="0.0 1.0 0.0"/>
 </joint>
-<ros2_control name="GazeboSystem" type="system">
-    <hardware>
-        <plugin>gazebo_ros2_control/GazeboSystem</plugin>
-    </hardware>
+<ros2_control name="RobotSystem" type="system">
+    <!-- ros2_control Gazebo -->
+    <xacro:if value="$(arg is_sim)">
+        <!-- ROS 2 Humble -->
+        <xacro:if value="$(arg is_ignition)">
+            <hardware><plugin>gz_ros2_control/GazeboSimSystem</plugin></hardware>
+        </xacro:if>
+        <!-- ROS 2 Iron or above -->
+        <xacro:unless value="$(arg is_ignition)">
+            <hardware><plugin>gz_ros2_control/GazeboSimSystem</plugin></hardware>
+        </xacro:unless>
+    </xacro:if>
+    <!-- ros2_control Real Robot (Placeholder) -->
+    <xacro:unless value="$(arg is_sim)">
+        <hardware><plugin>robotaksi_firmware/RobotaksiHardwareInterface</plugin></hardware>
+    </xacro:unless>
     <joint name="left_front_steering_joint">
         <command_interface name="position"/>
@@ -216,4 +230,5 @@
         <state_interface name="position"/>
         <state_interface name="velocity"/>
+        <param name="wheel_radius">${wheel_radius}</param>
     </joint>
     <joint name="right_back">
@@ -221,4 +236,5 @@
         <state_interface name="position"/>
         <state_interface name="velocity"/>
+        <param name="wheel_radius">${wheel_radius}</param>
     </joint>
 </ros2_control>
@@ -263,23 +279,4 @@
     </actuator>
 </transmission>
-<gazebo>
-    <plugin name="gazebo_ros2_control" filename="libgazebo_ros2_control.so">
-        <parameters>$(find robotaksi_controller)/config/controllers.yaml</parameters>
-    </plugin>
-</gazebo>
-<gazebo>
-    <plugin name="joint_state_publisher" filename="libgazebo_ros_joint_state_publisher.so">
-        <ros>
-            <remapping>~/out:=joint_states</remapping>
-        </ros>
-        <update_rate>30</update_rate>
-        <joint_name>left_front_steering_joint</joint_name>
-        <joint_name>right_front_steering_joint</joint_name>
-        <joint_name>left_front</joint_name>
-        <joint_name>right_front</joint_name>
-        <joint_name>left_back</joint_name>
-        <joint_name>right_back</joint_name>
-    </plugin>
-</gazebo>
 <xacro:rplidar_s2 parent="base_link" name="lidar" xyz="1.07 -0.015 0.63" rpy="0 0 0"/>
 <xacro:rplidar_s2_gazebo_plugin name="lidar"/>

File: robotaksi_description/urdf/rplidar_s2.xacro (robot description, xacro)
@@ -50,6 +50,8 @@
     <gazebo reference="${name}_laser_frame">
       <material>Gazebo/Black</material>
-      <sensor name="${name}_laser_sensor" type="ray">
+      <sensor name="${name}_laser_sensor" type="gpu_lidar">
         <pose>0 0 0 0 0 0</pose>
+        <topic>/scan</topic>
+        <update_rate>10.0</update_rate>
         <ray>
           <scan>
@@ -72,16 +74,5 @@
           </noise>
         </ray>
-        <update_rate>10.0</update_rate>
         <visualize>true</visualize>
-        <plugin name="${name}_laser_controller" filename="libgazebo_ros_ray_sensor.so">
-          <ros>
-            <remapping>~/out:=/scan</remapping>
-          </ros>
-          <output_type>sensor_msgs/LaserScan</output_type>
-          <frame_name>${name}_laser_frame</frame_name>
-          <min_range>0.2</min_range>
-          <max_range>20.0</max_range>
-          <range_resolution>0.02</range_resolution>
-        </plugin>
       </sensor>
     </gazebo>
