Commit message: display.launch düzeltildi

File: robotaksi_description/urdf/robotaksi.xacro (robot description, xacro)
@@ -21,5 +21,5 @@
   <inertial>
     <origin xyz="0.015227403646740032 -0.10161088779130478 0.2098030237602473" rpy="0 0 0"/>
-    <mass value="446.12211656731125"/>
+    <mass value="80"/>
     <inertia ixx="56.423509" iyy="169.853499" izz="202.959351" ixy="-0.254428" iyz="0.016951" ixz="0.803829"/>
   </inertial>

Commit message: igniton akerman entegre edildi

File: robotaksi_description/urdf/robotaksi.xacro (robot description, xacro)
@@ -159,5 +159,5 @@
     <origin xyz="0.725318 -0.705779 0.279785" rpy="0 0 0"/>
     <axis xyz="0 0 1"/>
-    <limit lower="-0.6" upper="0.6" effort="100" velocity="100"/>
+    <limit lower="-0.516" upper="0.516" effort="100" velocity="1"/>
 </joint>
 <joint name="left_front_steering_joint" type="revolute">
@@ -166,5 +166,5 @@
     <origin xyz="0.725318 0.50652 0.279262" rpy="0 0 0"/>
     <axis xyz="0 0 1"/>
-    <limit lower="-0.6" upper="0.6" effort="100" velocity="100"/>
+    <limit lower="-0.516" upper="0.516" effort="100" velocity="1"/>
 </joint>
 <joint name="right_front" type="continuous">
@@ -221,8 +221,10 @@
         <state_interface name="position"/>
         <state_interface name="velocity"/>
+        <param name="wheel_radius">${wheel_radius}</param>
     </joint>
     <joint name="right_front">
         <state_interface name="position"/>
         <state_interface name="velocity"/>
+        <param name="wheel_radius">${wheel_radius}</param>
     </joint>
     <joint name="left_back">
